File: DMX-Xi12/DMX-Xi12.kicad_pcb (KiCad board)
At the start: 2 copper layers, 177.8 x 200.7 mm, 189 parts, among them Con1 Cortex-10-SWD, Con10 Screw-terminal, Con2 Screw-terminal, Con3 Screw-terminal, Con4 Screw-terminal, Con5 Screw-terminal, Con6 Screw-terminal, Con7 Screw-terminal, Con8 Screw-terminal, Con9 Screw-terminal, J1 RJ45, J2 RJ45, P3 USB_B, SW1 Switch_SPDT_x2, SW2 DIPS_04, SW3 SW_PUSH, SW4 SW_PUSH, U1 MAX13450E, U10 BTA20, U11 BTA20, U12 BTA20, U13 BTA20, U14 AN-3003, U15 AN-3003, U16 AN-3003, U17 AN-3003, U18 BTA20, U19 BTA20, U2 LPC11U68JBD100E, U20 BTA20, U21 BTA20, U22 AN-3003, U23 AN-3003, U24 AN-3003, U25 AN-3003, U26 BTA20, U27 BTA20, U28 BTA20, U29 BTA20, U3 LTV-354T, U30 AN-3003, U31 AN-3003, U32 AN-3003, U33 AN-3003, U34 BTA20, U35 BTA20, U36 BTA20, U37 BTA20, U38 AN-3003, U39 AN-3003, U4 7805, U40 AN-3003, U41 AN-3003, U42 BTA20, U43 BTA20, U44 BTA20, U45 BTA20, U46 AN-3003, U47 AN-3003, U48 AN-3003, U49 AN-3003, U5 LTV-354T, U50 BTA20, U51 BTA20, U52 BTA20, U53 BTA20, U54 AN-3003, U55 AN-3003, U56 AN-3003, U57 AN-3003, U58 BTA20, U59 BTA20, U6 AN-3003, U60 BTA20, U61 BTA20, U62 AN-3003, U63 AN-3003, U64 AN-3003, U65 AN-3003, U66 BTA20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

Commit message: more work on board
Parts:
- added Con11: BARREL_JACK, Connect:BARREL_JACK, F.Cu at (233.7, 230.5)
- U4: value 7805 -> 7805n
- moved R2 231.9 mm to (120.0, 224.2), turned to 90 degrees
- moved R1 231.7 mm to (118.1, 225.4), turned to 90 degrees
- moved P3 229.0 mm to (120.0, 232.4), turned to 90 degrees
- moved J1 223.2 mm to (165.1, 229.2)
- moved Con9 182.7 mm to (234.9, 188.6), turned to 270 degrees
- moved U67 176.2 mm to (224.8, 196.2), turned to 90 degrees
- moved Con8 166.0 mm to (234.9, 158.1), turned to 270 degrees
- moved U66 164.9 mm to (224.8, 181.0), turned to 90 degrees
- moved Con6 164.3 mm to (234.9, 97.2), turned to 270 degrees
- moved U64 163.3 mm to (217.2, 191.1), turned to 270 degrees
- moved Con7 159.4 mm to (234.9, 127.6), turned to 270 degrees
- moved U69 156.2 mm to (207.0, 196.2), turned to 90 degrees
- moved U59 155.8 mm to (224.8, 165.7), turned to 90 degrees
- moved U65 153.8 mm to (217.2, 178.4), turned to 270 degrees
- moved U42 153.7 mm to (224.8, 89.5), turned to 90 degrees
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Connections:
- Con10 pad 1: /Power2/LiveB -> /Output1/LiveA
- Con10 pad 4: /Output1/LiveA -> /Power2/LiveB
- U10 pad 1: (no net) -> /Output1/LiveA
- U10 pad 2: (no net) -> /Output1/Live1
- U10 pad 3: (no net) -> Net-(U10-Pad3)
- U11 pad 1: (no net) -> /Output1/LiveA
- U11 pad 2: (no net) -> /Output1/Live2
- U11 pad 3: (no net) -> Net-(U11-Pad3)
- U12 pad 1: (no net) -> /Output1/LiveA
- U12 pad 2: (no net) -> /Output1/Live3
- U12 pad 3: (no net) -> Net-(U12-Pad3)
- U13 pad 1: (no net) -> /Output1/LiveA
- U13 pad 2: (no net) -> /Output1/Live4
- U13 pad 3: (no net) -> Net-(U13-Pad3)
- U18 pad 1: (no net) -> /Output1/LiveA
- U18 pad 2: (no net) -> /Output1/Live5
- U18 pad 3: (no net) -> Net-(U14-Pad4)
- U19 pad 1: (no net) -> /Output1/LiveA
- U19 pad 2: (no net) -> /Output1/Live6
- U19 pad 3: (no net) -> Net-(U15-Pad4)
- U20 pad 1: (no net) -> /Output1/LiveA
- U20 pad 2: (no net) -> /Output1/Live7
- U20 pad 3: (no net) -> Net-(U16-Pad4)
- U21 pad 1: (no net) -> /Output1/LiveA
- U21 pad 2: (no net) -> /Output1/Live8
- U21 pad 3: (no net) -> Net-(U17-Pad4)
- U26 pad 1: (no net) -> /Output1/LiveA
- U26 pad 2: (no net) -> /Output1/Live9
- U26 pad 3: (no net) -> Net-(U22-Pad4)
- U27 pad 1: (no net) -> /Output1/LiveA
- U27 pad 2: (no net) -> /Output1/Live10
- U27 pad 3: (no net) -> Net-(U23-Pad4)
- U28 pad 1: (no net) -> /Output1/LiveA
- U28 pad 2: (no net) -> /Output1/Live11
- U28 pad 3: (no net) -> Net-(U24-Pad4)
- U29 pad 1: (no net) -> /Output1/LiveA
- U29 pad 2: (no net) -> /Output1/Live12
- U29 pad 3: (no net) -> Net-(U25-Pad4)
- U34 pad 1: (no net) -> /Output1/LiveA
- U34 pad 2: (no net) -> /Output1/Live13
- U34 pad 3: (no net) -> Net-(U30-Pad4)
- U35 pad 1: (no net) -> /Output1/LiveA
- U35 pad 2: (no net) -> /Output1/Live14
- U35 pad 3: (no net) -> Net-(U31-Pad4)
- U36 pad 1: (no net) -> /Output1/LiveA
- U36 pad 2: (no net) -> /Output1/Live15
- U36 pad 3: (no net) -> Net-(U32-Pad4)
- U37 pad 1: (no net) -> /Output1/LiveA
- U37 pad 2: (no net) -> /Output1/Live16
- U37 pad 3: (no net) -> Net-(U33-Pad4)
- U4 pad 1: (no net) -> +5V
- U4 pad 2: (no net) -> GND
- U4 pad 3: (no net) -> +3V3
- U42 pad 1: (no net) -> /Power2/LiveB
- U42 pad 2: (no net) -> /Power2/Live17
- U42 pad 3: (no net) -> Net-(U38-Pad4)
- U43 pad 1: (no net) -> /Power2/LiveB
- U43 pad 2: (no net) -> /Power2/Live18
- U43 pad 3: (no net) -> Net-(U39-Pad4)
- U44 pad 1: (no net) -> /Power2/LiveB
- U44 pad 2: (no net) -> /Power2/Live19
- U44 pad 3: (no net) -> Net-(U40-Pad4)
- U45 pad 1: (no net) -> /Power2/LiveB
- U45 pad 2: (no net) -> /Power2/Live20
- U45 pad 3: (no net) -> Net-(U41-Pad4)
- U50 pad 1: (no net) -> /Power2/LiveB
- U50 pad 2: (no net) -> /Power2/Live21
- U50 pad 3: (no net) -> Net-(U46-Pad4)
- U51 pad 1: (no net) -> /Power2/LiveB
- U51 pad 2: (no net) -> /Power2/Live22
- U51 pad 3: (no net) -> Net-(U47-Pad4)
- U52 pad 1: (no net) -> /Power2/LiveB
- U52 pad 2: (no net) -> /Power2/Live23
- U52 pad 3: (no net) -> Net-(U48-Pad4)
- U53 pad 1: (no net) -> /Power2/LiveB
- U53 pad 2: (no net) -> /Power2/Live24
- U53 pad 3: (no net) -> Net-(U49-Pad4)
- U58 pad 1: (no net) -> /Power2/LiveB
- U58 pad 2: (no net) -> /Power2/Live25
- U58 pad 3: (no net) -> Net-(U54-Pad4)
- U59 pad 1: (no net) -> /Power2/LiveB
- U59 pad 2: (no net) -> /Power2/Live26
- U59 pad 3: (no net) -> Net-(U55-Pad4)
- U6 pad 4: Net-(U10-Pad~) -> Net-(U10-Pad3)
- U60 pad 1: (no net) -> /Power2/LiveB
- U60 pad 2: (no net) -> /Power2/Live27
- U60 pad 3: (no net) -> Net-(U56-Pad4)
- U61 pad 1: (no net) -> /Power2/LiveB
- U61 pad 2: (no net) -> /Power2/Live28
- U61 pad 3: (no net) -> Net-(U57-Pad4)
- U66 pad 1: (no net) -> /Power2/LiveB
- U66 pad 2: (no net) -> /Power2/Live29
- U66 pad 3: (no net) -> Net-(U62-Pad4)
- U67 pad 1: (no net) -> /Power2/LiveB
- U67 pad 2: (no net) -> /Power2/Live30
- U67 pad 3: (no net) -> Net-(U63-Pad4)
- U68 pad 1: (no net) -> /Power2/LiveB
- U68 pad 2: (no net) -> /Power2/Live31
- U68 pad 3: (no net) -> Net-(U64-Pad4)
- U69 pad 1: (no net) -> /Power2/LiveB
- U69 pad 2: (no net) -> /Power2/Live32
- U69 pad 3: (no net) -> Net-(U65-Pad4)
- U7 pad 4: Net-(U11-Pad~) -> Net-(U11-Pad3)
- U8 pad 4: Net-(U12-Pad~) -> Net-(U12-Pad3)
- U9 pad 4: Net-(U13-Pad~) -> Net-(U13-Pad3)
Routing:
- net +5V: track 0.00 -> 101.8 mm, vias 0 -> 2
- net +3V3: track 0.00 -> 75.2 mm
- net GND: track 0.00 -> 72.7 mm, vias 0 -> 13
- net Net-(R1-Pad2): track 0.00 -> 51.3 mm
- net Net-(R2-Pad2): track 0.00 -> 47.6 mm
- net Net-(J2-Pad1): track 0.00 -> 29.8 mm
- net Net-(J2-Pad2): track 0.00 -> 24.5 mm
- net Net-(J1-Pad1): track 0.00 -> 18.1 mm
- net Net-(C4-Pad1): track 0.00 -> 14.3 mm
- net Net-(C3-Pad1): track 0.00 -> 13.0 mm
- net Net-(J1-Pad2): track 0.00 -> 12.5 mm
- net /Front-End/RX: track 0.00 -> 4.79 mm
- net Net-(P3-Pad3): track 0.00 -> 4.06 mm
- net Net-(P3-Pad2): track 0.00 -> 3.24 mm
- net Net-(D2-Pad2): track 0.00 -> 2.95 mm
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- added copper zone on B.Cu, net GND
Other:
- board size 177.8 x 200.7 mm -> 177.8 x 177.8 mm
- net class Power added: clearance 0.2, trace_width 0.254, via_dia 0.6, via_drill 0.4

Commit message: completed board. Schematic, is correct but some part values and numbers need updating! Do not trust the schematic yet
Parts:
- removed C11: 0.01u, Capacitors_SMD:C_0603
- removed C13, C14, C15, C16, C17: 0.1u, Capacitors_SMD:C_0603
- removed R13, R14, R15, R7, R8, R9: 2k2, Resistors_SMD:R_0603
- added D3: LED, LEDs:LED_0603, F.Cu at (138.6, 208.8)
- added D4: D, Diodes_ThroughHole:Diode_DO-41_SOD81_Horizontal_RM10, F.Cu at (153.7, 226.7)
- added G***: LOGO, Components:Tep-silk, F.Cu at (152.4, 109.2)
- added G***: LOGO, Components:Tep-copper, F.Cu at (152.4, 109.2)
- added G***: LOGO, Components:Tep-soldermask, F.Cu at (152.4, 109.2)
- added R82: 330R, Resistors_SMD:R_0603, F.Cu at (142.2, 208.8)
- added R83: 10k, Resistors_SMD:R_0603, F.Cu at (135.9, 214.8)
- added R84: 10k, Resistors_SMD:R_0603, F.Cu at (139.1, 214.8)
- added REF**: 1pin, Connect:1pin, F.Cu at (81.0, 211.1)
- added REF**: 1pin, Connect:1pin, F.Cu at (81.0, 68.3)
- added REF**: 1pin, Connect:1pin, F.Cu at (223.8, 68.3)
- added REF**: 1pin, Connect:1pin, F.Cu at (223.8, 211.1)
- C12: value 0.1u -> 0.01u
- C9: value 4.7uF -> 1nF
- R12, R6: value 2k2 -> 100k
- U3, U5: value LTV-354T -> LTV-354T*
- moved R18 319.0 mm to (108.3, 234.9)
- moved R23 315.4 mm to (94.0, 222.9), turned to 270 degrees
- moved R22 312.4 mm to (94.0, 234.3), turned to 270 degrees
- moved R24 308.8 mm to (94.0, 211.5), turned to 270 degrees
- moved R19 304.4 mm to (108.3, 223.5)
- moved R20 303.2 mm to (108.3, 212.2)
- moved R25 302.4 mm to (94.0, 200.0), turned to 270 degrees
- moved R30 296.3 mm to (94.0, 188.6), turned to 270 degrees
- moved R21 290.8 mm to (108.3, 200.7)
- moved R31 290.6 mm to (94.0, 177.2), turned to 270 degrees
- moved R32 285.2 mm to (94.0, 165.7), turned to 270 degrees
- moved R26 284.5 mm to (108.3, 189.2)
- moved R33 280.2 mm to (94.0, 154.3), turned to 270 degrees
- moved R27 278.5 mm to (108.3, 177.8)
- moved R38 275.6 mm to (94.0, 142.9), turned to 270 degrees
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Connections:
- C8 pad 1: +3V3 -> GND
- C8 pad 2: GND -> +3V3
- Con10 pad 2: Net-(Con10-Pad2) -> /Power/Neutral
- Con10 pad 3: Net-(Con10-Pad3) -> /Earth
- Con10 pad 4: /Power2/LiveB -> /Power/LiveB
- P3 pad 4: GND -> Net-(P3-Pad4)
- R4 pad 1: Net-(R4-Pad1) -> Net-(Con1-Pad4)
- R53 pad 2: /Processor/CH19 -> /Power2/CH20
- R6 pad 1: /Power/LiveA -> /Output1/LiveA
- U1 pad 10: Net-(J2-Pad2) -> Net-(J2-Pad1)
- U1 pad 12: Net-(J2-Pad1) -> Net-(J2-Pad2)
- U1 pad 8: Net-(J1-Pad2) -> Net-(J1-Pad1)
- U1 pad 9: Net-(J1-Pad1) -> Net-(J1-Pad2)
- U2 pad 10: /Output1/CH8 -> /Output1/CH9
- U2 pad 100: /Power2/CH26 -> /Output1/CH11
- U2 pad 17: /Processor/RX -> /Front-End/RX
- U2 pad 18: /Output1/CH11 -> /Output1/CH8
- U2 pad 20: /Power2/CH27 -> /Output1/CH7
- U2 pad 22: /Power2/CH28 -> /Output1/CH6
- U2 pad 28: /Output1/CH2 -> /Output1/CH4
- U2 pad 29: /Power2/CH21 -> /Output1/CH3
- U2 pad 30: +3V3 -> Net-(R83-Pad2)
- U2 pad 33: /Processor/RX_ENABLE -> /Front-End/RX_ENABLE
- U2 pad 34: /Power2/CH18 -> /Output1/CH2
- U2 pad 35: /Power2/CH24 -> /Output1/CH1
- U2 pad 38: Net-(R2-Pad2) -> Net-(R1-Pad2)
- U2 pad 39: Net-(R1-Pad2) -> Net-(R2-Pad2)
- U2 pad 4: /Power2/CH19 -> /Output1/CH10
- U2 pad 42: /Power2/CH25 -> /Power2/CH32
- U2 pad 43: /Processor/CH19 -> /Power2/CH31
- U2 pad 46: /Power2/CH29 -> /Power2/CH30
- U2 pad 47: /Output1/CH6 -> /Power2/CH29
- U2 pad 48: /Power2/CH32 -> /Power2/CH28
- U2 pad 52: /Processor/Zero_crossingB -> /Power/Zero_crossingB
- U2 pad 55: /Output1/CH3 -> /Power2/CH27
- U2 pad 56: /Power2/CH22 -> /Power2/CH26
- U2 pad 57: /Processor/Zero_crossingA -> /Power/Zero_crossingA
- U2 pad 61: /Output1/CH9 -> /Power2/CH25
- U2 pad 62: /Processor/TX_ENABLE -> /Front-End/TX_ENABLE
- U2 pad 63: /Power2/CH30 -> /Power2/CH24
- U2 pad 65: /Output1/CH12 -> /Power2/CH23
- U2 pad 67: /Power2/CH31 -> /Power2/CH22
- U2 pad 72: /Output1/CH4 -> /Power2/CH21
- U2 pad 78: /Output1/CH14 -> /Power2/CH20
- U2 pad 79: /Output1/CH15 -> /Power2/CH19
- U2 pad 80: /Power2/CH23 -> /Power2/CH18
- U2 pad 81: Net-(U2-Pad81) -> Net-(Con1-Pad2)
- U2 pad 82: Net-(Con1-Pad2) -> Net-(U2-Pad82)
- U2 pad 86: /Output1/CH10 -> /Power2/CH17
- U2 pad 89: /Output1/CH13 -> /Output1/CH15
- U2 pad 96: /Power2/CH17 -> /Output1/CH14
- U2 pad 97: /Output1/CH1 -> /Output1/CH13
- U2 pad 98: /Output1/CH7 -> /Output1/CH12
- U3 pad 1: Net-(R9-Pad2) -> Net-(R6-Pad2)
- U3 pad 2: (no net) -> /Power/Neutral
- U3 pad 3: /Power/NeutralA -> GND
- U3 pad 4: GND -> /Power/Zero_crossingA
- U42 pad 1: /Power2/LiveB -> /Power/LiveB
- U43 pad 1: /Power2/LiveB -> /Power/LiveB
- U44 pad 1: /Power2/LiveB -> /Power/LiveB
- U45 pad 1: /Power2/LiveB -> /Power/LiveB
- U5 pad 1: Net-(R15-Pad2) -> Net-(R12-Pad2)
- U5 pad 2: (no net) -> /Power/Neutral
- U5 pad 3: /Power/NeutralB -> GND
- U5 pad 4: GND -> /Power/Zero_crossingB
- U50 pad 1: /Power2/LiveB -> /Power/LiveB
- U51 pad 1: /Power2/LiveB -> /Power/LiveB
- U52 pad 1: /Power2/LiveB -> /Power/LiveB
- U53 pad 1: /Power2/LiveB -> /Power/LiveB
- U58 pad 1: /Power2/LiveB -> /Power/LiveB
- U59 pad 1: /Power2/LiveB -> /Power/LiveB
- U60 pad 1: /Power2/LiveB -> /Power/LiveB
- U61 pad 1: /Power2/LiveB -> /Power/LiveB
- U66 pad 1: /Power2/LiveB -> /Power/LiveB
- U67 pad 1: /Power2/LiveB -> /Power/LiveB
- U68 pad 1: /Power2/LiveB -> /Power/LiveB
- U69 pad 1: /Power2/LiveB -> /Power/LiveB
Routing:
- net /Earth: track 0.00 -> 1177.0 mm, vias 0 -> 2
- net +3V3: track 75.2 -> 324.4 mm, vias 0 -> 4
- net /Power/Zero_crossingA: track 0.00 -> 170.8 mm, vias 0 -> 2
- net /Power2/CH17: track 0.00 -> 157.8 mm, vias 0 -> 2
- net /Power/Zero_crossingB: track 0.00 -> 155.2 mm, vias 0 -> 2
- net /Output1/CH16: track 0.00 -> 140.4 mm, vias 0 -> 2
- net /Power2/CH18: track 0.00 -> 138.3 mm, vias 0 -> 2
- net /Output1/CH15: track 0.00 -> 133.6 mm, vias 0 -> 2
- net /Power2/CH19: track 0.00 -> 126.5 mm, vias 0 -> 2
- net /Output1/CH14: track 0.00 -> 120.6 mm, vias 0 -> 2
- net /Power2/CH20: track 0.00 -> 114.4 mm, vias 0 -> 2
- net /Power2/CH21: track 0.00 -> 104.5 mm, vias 0 -> 2
- net /Output1/CH13: track 0.00 -> 104.1 mm, vias 0 -> 2
- net /Output1/CH12: track 0.00 -> 97.1 mm, vias 0 -> 2
- net /Power2/CH22: track 0.00 -> 95.8 mm, vias 0 -> 2
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- added copper zone on F.Cu, net /Output1/Live1
- added copper zone on F.Cu, net /Output1/Live10
- added copper zone on F.Cu, net /Output1/Live11
- added copper zone on F.Cu, net /Output1/Live12
- added copper zone on F.Cu, net /Output1/Live13
- added copper zone on F.Cu, net /Output1/Live14
- added copper zone on F.Cu, net /Output1/Live15
- added copper zone on F.Cu, net /Output1/Live16
- added copper zone on F.Cu, net /Output1/Live2
- added copper zone on F.Cu, net /Output1/Live3
- added copper zone on F.Cu, net /Output1/Live4
- added copper zone on F.Cu, net /Output1/Live5
- added copper zone on F.Cu, net /Output1/Live6
- added copper zone on F.Cu, net /Output1/Live7
- added copper zone on F.Cu, net /Output1/Live8
- added copper zone on F.Cu, net /Output1/Live9
- added copper zone on B.Cu, net /Output1/LiveA
- added copper zone on B.Cu, net /Power/LiveB
- added copper zone on F.Cu, net /Power2/Live17
- added copper zone on F.Cu, net /Power2/Live18
- added copper zone on F.Cu, net /Power2/Live19
- added copper zone on F.Cu, net /Power2/Live20
- added copper zone on F.Cu, net /Power2/Live21
- added copper zone on F.Cu, net /Power2/Live22
- added copper zone on F.Cu, net /Power2/Live23
- added copper zone on F.Cu, net /Power2/Live24
- added copper zone on F.Cu, net /Power2/Live25
- added copper zone on F.Cu, net /Power2/Live26
- added copper zone on F.Cu, net /Power2/Live27
- added copper zone on F.Cu, net /Power2/Live28
- added copper zone on F.Cu, net /Power2/Live29
- added copper zone on F.Cu, net /Power2/Live30
- added copper zone on F.Cu, net /Power2/Live31
- added copper zone on F.Cu, net /Power2/Live32
- added copper zone on F.Cu, net GND
Other:
- board size 177.8 x 177.8 mm -> 177.8 x 196.8 mm
- rule pad_to_mask_clearance: 0.2 -> 0.0762
- board text added: "5V"
- board text added: "Channel 1"
- board text added: "Channel 1 - PIO1_23 Channel 2 - PIO1_17 Channel 3 - PIO1_20 Channel 4 - PIO1_1 Channel 5 - PIO1_4 Channel 6 - PIO1_27 Channel 7 - PIO1_26 Channel 8 - PIO1_10 Channel 9 - PIO1_7 Channel 10 - PIO1_19 Channel 11 - PIO1_25 Channel 12 - PIO1_6 Channel 13 - PIO1_0 Channel 14 - PIO1_16 Channel 15 - PIO1_12 Channel 16 - PIO1_15 Channel 17 - PIO1_9 Channel 18 - PIO1_22 Channel 19 - PIO1_14 Channel 20 - PI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"
- board text added: "Channel 16"
- board text added: "Channel 17"
- board text added: "Channel 32"
- board text added: "DMX In"
- board text added: "DMX Out"
- board text added: "Earth"
- board text added: "Live A"
- board text added: "Live B"
- board text added: "Matt Hollands 05-2016 Matthew_Hollands@thcl.co.uk"
- board text added: "Neutral"
- board text added: "Tau Epsilon Phi Xi Chapter Lightshow 2016"
- board text added: "dlaw@dlaw.me"
