File: DMX-Xi12/Output1.sch (KiCad schematic (older format))
At the start: 48 parts

Commit message: more schematic
Parts:
- removed U? (x6): Live, symbol Live
Connections:
- net labels added: Live1, Live2, Live3, Live4, Live5, Live6
Changed lines of the file:
@@
 $Descr A4 11693 8268
 encoding utf-8
-Sheet 5 10
+Sheet 6 10
 Title ""
 Date ""
@@
 	3050 1550 3900 1550
 Wire Wire Line
-	4250 900  4250 1100
+	4250 750  4250 1100
 Wire Wire Line
 	3550 1500 3550 2100
@@
 Wire Wire Line
 	4250 2000 4250 2250
-$Comp
-L Live U?
-U 1 1 56B6AA9B
-P 4250 900
-F 0 "U?" H 4300 950 60  0000 C CNN
-F 1 "Live" H 4250 1150 60  0000 C CNN
-F 2 "" H 4250 900 60  0000 C CNN
-F 3 "" H 4250 900 60  0000 C CNN
-	1    4250 900
-	1    0    0    -1
-$EndComp
 Connection ~ 4250 1050
 Connection ~ 4250 2100
@@
 	3050 3650 3900 3650
 Wire Wire Line
-	4250 3000 4250 3200
+	4250 2900 4250 3200
 Wire Wire Line
 	3550 3600 3550 4200
@@
 Wire Wire Line
 	4250 4100 4250 4350
-$Comp
-L Live U?
-U 1 1 56B6B7A0
-P 4250 3000
-F 0 "U?" H 4300 3050 60  0000 C CNN
-F 1 "Live" H 4250 3250 60  0000 C CNN
-F 2 "" H 4250 3000 60  0000 C CNN
-F 3 "" H 4250 3000 60  0000 C CNN
-	1    4250 3000
-	1    0    0    -1
-$EndComp
 Connection ~ 4250 3150
 Connection ~ 4250 4200
@@
 	3050 5700 3900 5700
 Wire Wire Line
-	4250 5050 4250 5250
+	4250 4950 4250 5250
 Wire Wire Line
 	3550 5650 3550 6250
@@
 Wire Wire Line
 	4250 6150 4250 6400
-$Comp
-L Live U?
-U 1 1 56B6BA01
-P 4250 5050
-F 0 "U?" H 4300 5100 60  0000 C CNN
-F 1 "Live" H 4250 5300 60  0000 C CNN
-F 2 "" H 4250 5050 60  0000 C CNN
-F 3 "" H 4250 5050 60  0000 C CNN
-	1    4250 5050
-	1    0    0    -1
-$EndComp
 Connection ~ 4250 5200
 Connection ~ 4250 6250
@@
 	7050 1550 7900 1550
 Wire Wire Line
-	8250 900  8250 1100
+	8250 750  8250 1100
 Wire Wire Line
 	7550 1500 7550 2100
@@
 Wire Wire Line
 	8250 2000 8250 2250
-$Comp
-L Live U?
-U 1 1 56B6C132
-P 8250 900
-F 0 "U?" H 8300 950 60  0000 C CNN
-F 1 "Live" H 8250 1150 60  0000 C CNN
-F 2 "" H 8250 900 60  0000 C CNN
-F 3 "" H 8250 900 60  0000 C CNN
-	1    8250 900
-	1    0    0    -1
-$EndComp
 Connection ~ 8250 1050
 Connection ~ 8250 2100
@@
 	7050 3700 7900 3700
 Wire Wire Line
-	8250 3050 8250 3250
+	8250 2950 8250 3250
 Wire Wire Line
 	7550 3650 7550 4250
@@
 Wire Wire Line
 	8250 4150 8250 4400
-$Comp
-L Live U?
-U 1 1 56B6C463
-P 8250 3050
-F 0 "U?" H 8300 3100 60  0000 C CNN
-F 1 "Live" H 8250 3300 60  0000 C CNN
-F 2 "" H 8250 3050 60  0000 C CNN
-F 3 "" H 8250 3050 60  0000 C CNN
-	1    8250 3050
-	1    0    0    -1
-$EndComp
 Connection ~ 8250 3200
 Connection ~ 8250 4250
@@
 	7050 5650 7900 5650
 Wire Wire Line
-	8250 5000 8250 5200
+	8250 4950 8250 5200
 Wire Wire Line
 	7550 5600 7550 6200
@@
 Wire Wire Line
 	8250 6100 8250 6350
-$Comp
-L Live U?
-U 1 1 56B6C8D4
-P 8250 5000
-F 0 "U?" H 8300 5050 60  0000 C CNN
-F 1 "Live" H 8250 5250 60  0000 C CNN
-F 2 "" H 8250 5000 60  0000 C CNN
-F 3 "" H 8250 5000 60  0000 C CNN
-	1    8250 5000
-	1    0    0    -1
-$EndComp
 Connection ~ 8250 5150
 Connection ~ 8250 6200
@@
 	-1   0    0    1
 $EndComp
+Text Label 4250 750  1    60   ~ 0
+Live1
+Text Label 8250 750  1    60   ~ 0
+Live4
+Text Label 4250 2900 1    60   ~ 0
+Live2
+Text Label 8250 2950 1    60   ~ 0
+Live5
+Text Label 4250 4950 1    60   ~ 0
+Live3
+Text Label 8250 4950 1    60   ~ 0
+Live6
 $EndSCHEMATC

Commit message: made dlaw changes etc
Parts:
- removed C? (x6): 0.3u, symbol C
- removed R? (x6): 200R, symbol R
- removed R? (x6): 180R, symbol R
- removed R? (x6): 800R, symbol R
- removed U? (x6): AN-3003, symbol AN-3003
- removed U? (x6): BTA20, symbol BTA20
- removed U? (x6): Neutral, symbol Neutral
- added R? (x16): 200R, symbol R
- added R? (x16): 180R, symbol R
- added U? (x16): AN-3003, symbol AN-3003
- added U? (x16): BTA20, symbol BTA20
Connections:
- net labels added: CH10, CH11, CH12, CH13, CH14, CH15, CH16, CH7, CH8, CH9, Live10, Live11, Live12, Live13, Live14, Live15, Live16, Live7, Live8, Live9, NeutralA
- wire segments 78 -> 144
- no-connect marks 12 -> 32

Commit message: working on pcb
Parts:
- R18, R19, R20, R21, R22, R23, R24, R25, R26, R27, R28, R29, R30, R31, R32, R33, R34, R35, R36, R37, R38, R39, R40, R41, R42, R43, R44, R45, R46, R47, R48, R49: renamed from R?; footprint (none) -> Resistors_SMD:R_0603
- U10, U11, U12, U13, U18, U19, U20, U21, U26, U27, U28, U29, U34, U35, U36, U37: renamed from U?; footprint (none) -> Power_Integrations:TO-220
- U14, U15, U16, U17, U22, U23, U24, U25, U30, U31, U32, U33, U6, U7, U8, U9: renamed from U?; footprint (none) -> Housings_DIP:DIP-6_W7.62mm_LongPads
Connections:
- net NeutralA renamed LiveA
