File: DMX-Xi12/Power.sch (KiCad schematic (older format))
At the start: 3 parts

Commit message: more schematic
Parts:
- added D? (x2): LED, symbol LED
- added R?: 390, symbol R
- added R?: 220, symbol R
- added R?: 1k, symbol R
- added R? (x3): 2k7, symbol R
- added U?: LTV-354T, MFSOP-6, symbol LTV-354T
- added U?: Live, symbol Live
- added U?: Neutral, symbol Neutral
Connections:
- net labels added: Zero_crossing
- wire segments 8 -> 24
Changed lines of the file:
@@
 	1    0    0    -1
 $EndComp
-Wire Wire Line
-	4300 1500 4750 1500
 $Comp
 L GND #PWR?
@@
 	1    0    0    -1
 $EndComp
-Wire Wire Line
-	5150 2200 5150 1800
 $Comp
 L C C?
@@
 	1    0    0    -1
 $EndComp
-Wire Wire Line
-	4700 1700 4700 1500
-Connection ~ 4700 1500
-Wire Wire Line
-	4700 2000 4700 2100
-Wire Wire Line
-	4700 2100 5600 2100
-Connection ~ 5150 2100
-Wire Wire Line
-	5600 2100 5600 2000
-Wire Wire Line
-	5600 1700 5600 1500
-Wire Wire Line
-	5550 1500 5900 1500
 $Comp
 L +3.3V #PWR?
@@
 	1    0    0    -1
 $EndComp
+$Comp
+L LED D?
+U 1 1 56CBF4BA
+P 2900 1850
+F 0 "D?" H 2900 1950 50  0000 C CNN
+F 1 "LED" H 2900 1750 50  0000 C CNN
+F 2 "" H 2900 1850 50  0000 C CNN
+F 3 "" H 2900 1850 50  0000 C CNN
+	1    2900 1850
+	0    -1   -1   0
+$EndComp
+$Comp
+L +5V #PWR?
+U 1 1 56CBF4F1
+P 2900 1000
+F 0 "#PWR?" H 2900 850 50  0001 C CNN
+F 1 "+5V" H 2900 1140 50  0000 C CNN
+F 2 "" H 2900 1000 50  0000 C CNN
+F 3 "" H 2900 1000 50  0000 C CNN
+	1    2900 1000
+	1    0    0    -1
+$EndComp
+$Comp
+L GND #PWR?
+U 1 1 56CBF50D
+P 2900 2200
+F 0 "#PWR?" H 2900 1950 50  0001 C CNN
+F 1 "GND" H 2900 2050 50  0000 C CNN
+F 2 "" H 2900 2200 50  0000 C CNN
+F 3 "" H 2900 2200 50  0000 C CNN
+	1    2900 2200
+	1    0    0    -1
+$EndComp
+$Comp
+L R R?
+U 1 1 56CBF547
+P 2900 1300
+F 0 "R?" V 2980 1300 50  0000 C CNN
+F 1 "390" V 2900 1300 50  0000 C CNN
+F 2 "" V 2830 1300 50  0000 C CNN
+F 3 "" H 2900 1300 50  0000 C CNN
+	1    2900 1300
+	1    0    0    -1
+$EndComp
+$Comp
+L LED D?
+U 1 1 56CBF928
+P 6900 1850
+F 0 "D?" H 6900 1950 50  0000 C CNN
+F 1 "LED" H 6900 1750 50  0000 C CNN
+F 2 "" H 6900 1850 50  0000 C CNN
+F 3 "" H 6900 1850 50  0000 C CNN
+	1    6900 1850
+	0    -1   -1   0
+$EndComp
+$Comp
+L GND #PWR?
+U 1 1 56CBF934
+P 6900 2200
+F 0 "#PWR?" H 6900 1950 50  0001 C CNN
+F 1 "GND" H 6900 2050 50  0000 C CNN
+F 2 "" H 6900 2200 50  0000 C CNN
+F 3 "" H 6900 2200 50  0000 C CNN
+	1    6900 2200
+	1    0    0    -1
+$EndComp
+$Comp
+L R R?
+U 1 1 56CBF93A
+P 6900 1300
+F 0 "R?" V 6980 1300 50  0000 C CNN
+F 1 "220" V 6900 1300 50  0000 C CNN
+F 2 "" V 6830 1300 50  0000 C CNN
+F 3 "" H 6900 1300 50  0000 C CNN
+	1    6900 1300
+	1    0    0    -1
+$EndComp
+$Comp
+L +3.3V #PWR?
+U 1 1 56CBF969
+P 6900 1000
+F 0 "#PWR?" H 6900 850 50  0001 C CNN
+F 1 "+3.3V" H 6900 1140 50  0000 C CNN
+F 2 "" H 6900 1000 50  0000 C CNN
+F 3 "" H 6900 1000 50  0000 C CNN
+	1    6900 1000
+	1    0    0    -1
+$EndComp
+$Comp
+L LTV-354T U?
+U 1 1 56CCBACF
+P 2850 4850
+F 0 "U?" H 2640 5040 50  0000 L CNN
+F 1 "LTV-354T" H 2850 5050 50  0000 L CNN
+F 2 "MFSOP-6" H 2650 4650 50  0000 L CIN
+F 3 "" H 2875 4850 50  0000 L CNN
+	1    2850 4850
+	1    0    0    -1
+$EndComp
+$Comp
+L Live U?
+U 1 1 56CCBD8E
+P 2300 3450
+F 0 "U?" H 2350 3500 60  0000 C CNN
+F 1 "Live" H 2300 3700 60  0000 C CNN
+F 2 "" H 2300 3450 60  0000 C CNN
+F 3 "" H 2300 3450 60  0000 C CNN
+	1    2300 3450
+	1    0    0    -1
+$EndComp
+$Comp
+L Neutral U?
+U 1 1 56CCBDCB
+P 2300 5200
+F 0 "U?" H 2550 5400 60  0000 C CNN
+F 1 "Neutral" H 2300 5450 60  0000 C CNN
+F 2 "" H 2300 5200 60  0000 C CNN
+F 3 "" H 2300 5200 60  0000 C CNN
+	1    2300 5200
+	-1   0    0    1
+$EndComp
+$Comp
+L R R?
+U 1 1 56CCBE6A
+P 3150 4350
+F 0 "R?" V 3230 4350 50  0000 C CNN
+F 1 "1k" V 3150 4350 50  0000 C CNN
+F 2 "" V 3080 4350 50  0000 C CNN
+F 3 "" H 3150 4350 50  0000 C CNN
+	1    3150 4350
+	1    0    0    -1
+$EndComp
+$Comp
+L +3.3V #PWR?
+U 1 1 56CCBF90
+P 3150 4050
+F 0 "#PWR?" H 3150 3900 50  0001 C CNN
+F 1 "+3.3V" H 3150 4190 50  0000 C CNN
+F 2 "" H 3150 4050 50  0000 C CNN
+F 3 "" H 3150 4050 50  0000 C CNN
+	1    3150 4050
+	1    0    0    -1
+$EndComp
+$Comp
+L GND #PWR?
+U 1 1 56CCC098
+P 3150 5250
+F 0 "#PWR?" H 3150 5000 50  0001 C CNN
+F 1 "GND" H 3150 5100 50  0000 C CNN
+F 2 "" H 3150 5250 50  0000 C CNN
+F 3 "" H 3150 5250 50  0000 C CNN
+	1    3150 5250
+	1    0    0    -1
+$EndComp
+$Comp
+L R R?
+U 1 1 56CCC1C9
+P 2300 4600
+F 0 "R?" V 2380 4600 50  0000 C CNN
+F 1 "2k7" V 2300 4600 50  0000 C CNN
+F 2 "" V 2230 4600 50  0000 C CNN
+F 3 "" H 2300 4600 50  0000 C CNN
+	1    2300 4600
+	1    0    0    -1
+$EndComp
+$Comp
+L R R?
+U 1 1 56CCC234
+P 2300 4250
+F 0 "R?" V 2380 4250 50  0000 C CNN
+F 1 "2k7" V 2300 4250 50  0000 C CNN
+F 2 "" V 2230 4250 50  0000 C CNN
+F 3 "" H 2300 4250 50  0000 C CNN
+	1    2300 4250
+	1    0    0    -1
+$EndComp
+$Comp
+L R R?
+U 1 1 56CCC289
+P 2300 3900
+F 0 "R?" V 2380 3900 50  0000 C CNN
+F 1 "2k7" V 2300 3900 50  0000 C CNN
+F 2 "" V 2230 3900 50  0000 C CNN
+F 3 "" H 2300 3900 50  0000 C CNN
+	1    2300 3900
+	1    0    0    -1
+$EndComp
+Wire Wire Line
+	4300 1500 4750 1500
+Wire Wire Line
+	5150 1800 5150 2200
+Wire Wire Line
+	4700 1700 4700 1500
+Connection ~ 4700 1500
+Wire Wire Line
+	4700 2000 4700 2100
+Wire Wire Line
+	4700 2100 5600 2100
+Connection ~ 5150 2100
+Wire Wire Line
+	5600 2100 5600 2000
+Wire Wire Line
+	5600 1700 5600 1500
+Wire Wire Line
+	5550 1500 5900 1500
 Connection ~ 5600 1500
+Wire Wire Line
+	2900 1150 2900 1000
+Wire Wire Line
+	2900 1450 2900 1650
+Wire Wire Line
+	2900 2050 2900 2200
+Wire Wire Line
+	6900 1150 6900 1000
+Wire Wire Line
+	6900 1450 6900 1650
+Wire Wire Line
+	6900 2050 6900 2200
+Wire Wire Line
+	3150 4050 3150 4200
+Wire Wire Line
+	3150 4500 3150 4750
+Wire Wire Line
+	3150 5250 3150 4950
+Wire Wire Line
+	2300 5200 2300 4950
+Wire Wire Line
+	2300 4950 2550 4950
+Wire Wire Line
+	2550 4750 2300 4750
+Wire Wire Line
+	2300 3750 2300 3450
+Wire Wire Line
+	2300 4050 2300 4100
+Wire Wire Line
+	2300 4400 2300 4450
+Text HLabel 3450 4550 2    60   Output ~ 0
+Zero_crossing
+Wire Wire Line
+	3450 4550 3150 4550
+Connection ~ 3150 4550
 $EndSCHEMATC

Commit message: changed processor to 3.3v and added programming
Changed lines of the file:
@@
-$EndComp
-$Comp
-L +3.3V #PWR?
-U 1 1 56CCBF90
-P 3150 4050
-F 0 "#PWR?" H 3150 3900 50  0001 C CNN
-F 1 "+3.3V" H 3150 4190 50  0000 C CNN
-F 2 "" H 3150 4050 50  0000 C CNN
-F 3 "" H 3150 4050 50  0000 C CNN
-	1    3150 4050
-	1    0    0    -1
 $EndComp
 $Comp
@@
 	6900 2050 6900 2200
 Wire Wire Line
-	3150 4050 3150 4200
+	3150 4000 3150 4200
 Wire Wire Line
 	3150 4500 3150 4750
@@
 	3450 4550 3150 4550
 Connection ~ 3150 4550
+$Comp
+L +5V #PWR?
+U 1 1 56CD2B25
+P 3150 4000
+F 0 "#PWR?" H 3150 3850 50  0001 C CNN
+F 1 "+5V" H 3150 4140 50  0000 C CNN
+F 2 "" H 3150 4000 50  0000 C CNN
+F 3 "" H 3150 4000 50  0000 C CNN
+	1    3150 4000
+	1    0    0    -1
+$EndComp
 $EndSCHEMATC

Commit message: made dlaw changes etc
Parts:
- removed U?: Live, symbol Live
- removed U?: Neutral, symbol Neutral
- added R? (x5): 2k2, symbol R
- added R?: 1k, symbol R
- added U?: LTV-354T, MFSOP-6, symbol LTV-354T
- R? (x3): value 2k7 -> 2k2
Connections:
- net labels added: LiveA, LiveB, NeutralA, NeutralB, Zero_crossingA, Zero_crossingB
- net labels removed: Zero_crossing
- wire segments 24 -> 36
Other:
- moved on the sheet: C?, D?, R?, U?

Commit message: working on pcb
Parts:
- removed U?: LM1084IS-3.3/NOPB, TO-263, symbol LM1084IS-3.3/NOPB
- added U4: 7805, TO_SOT_Packages_SMD:TO-252-2Lead, symbol 7805
- C18, C19: renamed from C?; footprint (none) -> Capacitors_SMD:C_0603
- D1, D2: renamed from D?; footprint (none) -> LEDs:LED_0603
- R10, R11, R12, R13, R14, R15, R16, R17, R6, R7, R8, R9: renamed from R?; footprint (none) -> Resistors_SMD:R_0603
- U3, U5: renamed from U?; footprint MFSOP-6 -> Opto-Devices:Optocoupler_SMD_HandSoldering_KPC357_LTV35x_PC357_SingleChannel
Connections:
- net +3V3: now also U4.VO
- net +5V: now also U4.VI
- net GND: now also U4.GND
Changed lines of the file:
@@
 $EndDescr
 $Comp
-L LM1084IS-3.3/NOPB U?
-U 1 1 56B68233
-P 3450 1500
-F 0 "U?" H 3650 1300 50  0000 C CNN
-F 1 "LM1084IS-3.3/NOPB" H 3150 1700 50  0000 L CNN
-F 2 "TO-263" H 3450 1600 50  0000 C CIN
-F 3 "" H 3450 1500 50  0000 C CNN
-	1    3450 1500
-	1    0    0    -1
-$EndComp
-$Comp
-L +5V #PWR?
+L +5V #PWR029
 U 1 1 56B6829F
 P 2600 1450
-F 0 "#PWR?" H 2600 1300 50  0001 C CNN
+F 0 "#PWR029" H 2600 1300 50  0001 C CNN
 F 1 "+5V" H 2600 1590 50  0000 C CNN
 F 2 "" H 2600 1450 50  0000 C CNN
@@
 $EndComp
 $Comp
-L GND #PWR?
+L GND #PWR030
 U 1 1 56B682B8
 P 3450 2150
-F 0 "#PWR?" H 3450 1900 50  0001 C CNN
+F 0 "#PWR030" H 3450 1900 50  0001 C CNN
 F 1 "GND" H 3450 2000 50  0000 C CNN
 F 2 "" H 3450 2150 50  0000 C CNN
@@
 $EndComp
 $Comp
-L C C?
+L C C18
 U 1 1 56B682D2
 P 3000 1800
-F 0 "C?" H 3025 1900 50  0000 L CNN
+F 0 "C18" H 3025 1900 50  0000 L CNN
 F 1 "10u" H 3025 1700 50  0000 L CNN
-F 2 "" H 3038 1650 50  0000 C CNN
+F 2 "Capacitors_SMD:C_0603" H 3038 1650 50  0001 C CNN
 F 3 "" H 3000 1800 50  0000 C CNN
 	1    3000 1800
@@
 $EndComp
 $Comp
-L C C?
+L C C19
 U 1 1 56B68303
 P 3900 1800
-F 0 "C?" H 3925 1900 50  0000 L CNN
+F 0 "C19" H 3925 1900 50  0000 L CNN
 F 1 "10u" H 3925 1700 50  0000 L CNN
-F 2 "" H 3938 1650 50  0000 C CNN
+F 2 "Capacitors_SMD:C_0603" H 3938 1650 50  0001 C CNN
 F 3 "" H 3900 1800 50  0000 C CNN
 	1    3900 1800
@@
 $EndComp
 $Comp
-L +3.3V #PWR?
+L +3.3V #PWR031
 U 1 1 56B6835A
 P 4200 1450
-F 0 "#PWR?" H 4200 1300 50  0001 C CNN
+F 0 "#PWR031" H 4200 1300 50  0001 C CNN
 F 1 "+3.3V" H 4200 1590 50  0000 C CNN
 F 2 "" H 4200 1450 50  0000 C CNN
@@
 $EndComp
 $Comp
-L LED D?
+L LED D1
 U 1 1 56CBF4BA
 P 1200 1800
-F 0 "D?" H 1200 1900 50  0000 C CNN
+F 0 "D1" H 1200 1900 50  0000 C CNN
 F 1 "LED" H 1200 1700 50  0000 C CNN
-F 2 "" H 1200 1800 50  0000 C CNN
+F 2 "LEDs:LED_0603" H 1200 1600 50  0000 C CNN
 F 3 "" H 1200 1800 50  0000 C CNN
 	1    1200 1800
@@
 $EndComp
 $Comp
-L +5V #PWR?
+L +5V #PWR032
 U 1 1 56CBF4F1
 P 1200 950
-F 0 "#PWR?" H 1200 800 50  0001 C CNN
+F 0 "#PWR032" H 1200 800 50  0001 C CNN
 F 1 "+5V" H 1200 1090 50  0000 C CNN
 F 2 "" H 1200 950 50  0000 C CNN
@@
 $EndComp
 $Comp
-L GND #PWR?
+L GND #PWR033
 U 1 1 56CBF50D
 P 1200 2150
-F 0 "#PWR?" H 1200 1900 50  0001 C CNN
+F 0 "#PWR033" H 1200 1900 50  0001 C CNN
 F 1 "GND" H 1200 2000 50  0000 C CNN
 F 2 "" H 1200 2150 50  0000 C CNN
@@
 $EndComp
 $Comp
-L R R?
+L R R10
 U 1 1 56CBF547
 P 1200 1250
-F 0 "R?" V 1280 1250 50  0000 C CNN
+F 0 "R10" V 1280 1250 50  0000 C CNN
 F 1 "390" V 1200 1250 50  0000 C CNN
-F 2 "" V 1130 1250 50  0000 C CNN
+F 2 "Resistors_SMD:R_0603" V 1050 1250 50  0000 C CNN
 F 3 "" H 1200 1250 50  0000 C CNN
 	1    1200 1250
@@
 $EndComp
 $Comp
-L LED D?
+L LED D2
 U 1 1 56CBF928
 P 5200 1800
-F 0 "D?" H 5200 1900 50  0000 C CNN
+F 0 "D2" H 5200 1900 50  0000 C CNN
 F 1 "LED" H 5200 1700 50  0000 C CNN
-F 2 "" H 5200 1800 50  0000 C CNN
+F 2 "LEDs:LED_0603" H 5200 1800 50  0001 C CNN
 F 3 "" H 5200 1800 50  0000 C CNN
 	1    5200 1800
@@
 $EndComp
 $Comp
-L GND #PWR?
+L GND #PWR034
 U 1 1 56CBF934
 P 5200 2150
-F 0 "#PWR?" H 5200 1900 50  0001 C CNN
+F 0 "#PWR034" H 5200 1900 50  0001 C CNN
 F 1 "GND" H 5200 2000 50  0000 C CNN
 F 2 "" H 5200 2150 50  0000 C CNN
@@
 $EndComp
 $Comp
-L R R?
+L R R17
 U 1 1 56CBF93A
 P 5200 1250
-F 0 "R?" V 5280 1250 50  0000 C CNN
+F 0 "R17" V 5280 1250 50  0000 C CNN
 F 1 "220" V 5200 1250 50  0000 C CNN
-F 2 "" V 5130 1250 50  0000 C CNN
+F 2 "Resistors_SMD:R_0603" V 5130 1250 50  0001 C CNN
 F 3 "" H 5200 1250 50  0000 C CNN
 	1    5200 1250
@@
 $EndComp
 $Comp
-L +3.3V #PWR?
+L +3.3V #PWR035
 U 1 1 56CBF969
 P 5200 950
-F 0 "#PWR?" H 5200 800 50  0001 C CNN
+F 0 "#PWR035" H 5200 800 50  0001 C CNN
 F 1 "+3.3V" H 5200 1090 50  0000 C CNN
 F 2 "" H 5200 950 50  0000 C CNN
@@
 $EndComp
 $Comp
-L LTV-354T U?
+L LTV-354T U3
 U 1 1 56CCBACF
 P 1450 6650
-F 0 "U?" H 1240 6840 50  0000 L CNN
+F 0 "U3" H 1240 6840 50  0000 L CNN
 F 1 "LTV-354T" H 1450 6850 50  0000 L CNN
-F 2 "MFSOP-6" H 1250 6450 50  0000 L CIN
+F 2 "Opto-Devices:Optocoupler_SMD_HandSoldering_KPC357_LTV35x_PC357_SingleChannel" H 1250 6450 50  0000 L CIN
 F 3 "" H 1475 6650 50  0000 L CNN
 	1    1450 6650
@@
 $EndComp
 $Comp
-L R R?
+L R R11
 U 1 1 56CCBE6A
 P 1750 6150
-F 0 "R?" V 1830 6150 50  0000 C CNN
+F 0 "R11" V 1830 6150 50  0000 C CNN
 F 1 "1k" V 1750 6150 50  0000 C CNN
-F 2 "" V 1680 6150 50  0000 C CNN
+F 2 "Resistors_SMD:R_0603" V 1680 6150 50  0001 C CNN
 F 3 "" H 1750 6150 50  0000 C CNN
 	1    1750 6150
@@
 $EndComp
 $Comp
-L GND #PWR?
+L GND #PWR036
 U 1 1 56CCC098
 P 1750 7050
-F 0 "#PWR?" H 1750 6800 50  0001 C CNN
+F 0 "#PWR036" H 1750 6800 50  0001 C CNN
 F 1 "GND" H 1750 6900 50  0000 C CNN
 F 2 "" H 1750 7050 50  0000 C CNN
@@
 $EndComp
 $Comp
-L R R?
+L R R9
 U 1 1 56CCC1C9
 P 900 6400
-F 0 "R?" V 980 6400 50  0000 C CNN
+F 0 "R9" V 980 6400 50  0000 C CNN
 F 1 "2k2" V 900 6400 50  0000 C CNN
-F 2 "" V 830 6400 50  0000 C CNN
+F 2 "Resistors_SMD:R_0603" V 830 6400 50  0001 C CNN
 F 3 "" H 900 6400 50  0000 C CNN
 	1    900  6400
@@
 $EndComp
 $Comp
-L R R?
+L R R8
 U 1 1 56CCC234
 P 900 6050
-F 0 "R?" V 980 6050 50  0000 C CNN
+F 0 "R8" V 980 6050 50  0000 C CNN
 F 1 "2k2" V 900 6050 50  0000 C CNN
-F 2 "" V 830 6050 50  0000 C CNN
+F 2 "Resistors_SMD:R_0603" V 830 6050 50  0001 C CNN
 F 3 "" H 900 6050 50  0000 C CNN
 	1    900  6050
@@
 $EndComp
 $Comp
-L R R?
+L R R7
 U 1 1 56CCC289
 P 900 5700
-F 0 "R?" V 980 5700 50  0000 C CNN
+F 0 "R7" V 980 5700 50  0000 C CNN
 F 1 "2k2" V 900 5700 50  0000 C CNN
-F 2 "" V 830 5700 50  0000 C CNN
+F 2 "Resistors_SMD:R_0603" V 830 5700 50  0001 C CNN
 F 3 "" H 900 5700 50  0000 C CNN
 	1    900  5700
@@
 Connection ~ 1750 6350
 $Comp
-L R R?
+L R R6
 U 1 1 56D29409
 P 900 5350
-F 0 "R?" V 980 5350 50  0000 C CNN
+F 0 "R6" V 980 5350 50  0000 C CNN
 F 1 "2k2" V 900 5350 50  0000 C CNN
-F 2 "" V 830 5350 50  0000 C CNN
+F 2 "Resistors_SMD:R_0603" V 830 5350 50  0000 C CNN
 F 3 "" H 900 5350 50  0000 C CNN
 	1    900  5350
@@
 	900  4900 900  5200
 $Comp
-L LTV-354T U?
+L LTV-354T U5
 U 1 1 56D2988E
 P 3700 6650
-F 0 "U?" H 3490 6840 50  0000 L CNN
+F 0 "U5" H 3490 6840 50  0000 L CNN
 F 1 "LTV-354T" H 3700 6850 50  0000 L CNN
-F 2 "MFSOP-6" H 3500 6450 50  0000 L CIN
+F 2 "Opto-Devices:Optocoupler_SMD_HandSoldering_KPC357_LTV35x_PC357_SingleChannel" H 3500 6450 50  0000 L CIN
 F 3 "" H 3725 6650 50  0000 L CNN
 	1    3700 6650
@@
 $EndComp
 $Comp
-L R R?
+L R R16
 U 1 1 56D298A0
 P 4000 6150
-F 0 "R?" V 4080 6150 50  0000 C CNN
+F 0 "R16" V 4080 6150 50  0000 C CNN
 F 1 "1k" V 4000 6150 50  0000 C CNN
-F 2 "" V 3930 6150 50  0000 C CNN
+F 2 "Resistors_SMD:R_0603" V 3930 6150 50  0001 C CNN
 F 3 "" H 4000 6150 50  0000 C CNN
 	1    4000 6150
@@
 $EndComp
 $Comp
-L GND #PWR?
+L GND #PWR037
 U 1 1 56D298A6
 P 4000 7050
-F 0 "#PWR?" H 4000 6800 50  0001 C CNN
+F 0 "#PWR037" H 4000 6800 50  0001 C CNN
 F 1 "GND" H 4000 6900 50  0000 C CNN
 F 2 "" H 4000 7050 50  0000 C CNN
@@
 $EndComp
 $Comp
-L R R?
+L R R15
 U 1 1 56D298AC
 P 3150 6400
-F 0 "R?" V 3230 6400 50  0000 C CNN
+F 0 "R15" V 3230 6400 50  0000 C CNN
 F 1 "2k2" V 3150 6400 50  0000 C CNN
-F 2 "" V 3080 6400 50  0000 C CNN
+F 2 "Resistors_SMD:R_0603" V 3080 6400 50  0001 C CNN
 F 3 "" H 3150 6400 50  0000 C CNN
 	1    3150 6400
@@
 $EndComp
 $Comp
-L R R?
+L R R14
 U 1 1 56D298B2
 P 3150 6050
-F 0 "R?" V 3230 6050 50  0000 C CNN
+F 0 "R14" V 3230 6050 50  0000 C CNN
 F 1 "2k2" V 3150 6050 50  0000 C CNN
-F 2 "" V 3080 6050 50  0000 C CNN
+F 2 "Resistors_SMD:R_0603" V 3080 6050 50  0001 C CNN
 F 3 "" H 3150 6050 50  0000 C CNN
 	1    3150 6050
@@
 $EndComp
 $Comp
-L R R?
+L R R13
 U 1 1 56D298B8
 P 3150 5700
-F 0 "R?" V 3230 5700 50  0000 C CNN
+F 0 "R13" V 3230 5700 50  0000 C CNN
 F 1 "2k2" V 3150 5700 50  0000 C CNN
-F 2 "" V 3080 5700 50  0000 C CNN
+F 2 "Resistors_SMD:R_0603" V 3080 5700 50  0001 C CNN
 F 3 "" H 3150 5700 50  0000 C CNN
 	1    3150 5700
@@
 Connection ~ 4000 6350
 $Comp
-L R R?
+L R R12
 U 1 1 56D298CF
 P 3150 5350
-F 0 "R?" V 3230 5350 50  0000 C CNN
+F 0 "R12" V 3230 5350 50  0000 C CNN
 F 1 "2k2" V 3150 5350 50  0000 C CNN
-F 2 "" V 3080 5350 50  0000 C CNN
+F 2 "Resistors_SMD:R_0603" V 3080 5350 50  0001 C CNN
 F 3 "" H 3150 5350 50  0000 C CNN
 	1    3150 5350
@@
 LiveB
 $Comp
-L +3.3V #PWR?
+L +3.3V #PWR038
 U 1 1 56D2A01A
 P 1750 5800
-F 0 "#PWR?" H 1750 5650 50  0001 C CNN
+F 0 "#PWR038" H 1750 5650 50  0001 C CNN
 F 1 "+3.3V" H 1750 5940 50  0000 C CNN
 F 2 "" H 1750 5800 50  0000 C CNN
@@
 $EndComp
 $Comp
-L +3.3V #PWR?
+L +3.3V #PWR039
 U 1 1 56D2A058
 P 4000 5800
-F 0 "#PWR?" H 4000 5650 50  0001 C CNN
+F 0 "#PWR039" H 4000 5650 50  0001 C CNN
 F 1 "+3.3V" H 4000 5940 50  0000 C CNN
 F 2 "" H 4000 5800 50  0000 C CNN
@@
 Text HLabel 3150 7100 3    60   Input ~ 0
 NeutralB
+$Comp
+L 7805 U4
+U 1 1 570B82C2
+P 3450 1500
+F 0 "U4" H 3600 1304 50  0000 C CNN
+F 1 "7805" H 3450 1700 50  0000 C CNN
+F 2 "TO_SOT_Packages_SMD:TO-252-2Lead" H 3450 1500 50  0001 C CNN
+F 3 "" H 3450 1500 50  0000 C CNN
+	1    3450 1500
+	1    0    0    -1
+$EndComp
 $EndSCHEMATC

Commit message: more work on board
Parts:
- removed U4: 7805, TO_SOT_Packages_SMD:TO-252-2Lead, symbol 7805
- added Con11: BARREL_JACK, Connect:BARREL_JACK, symbol BARREL_JACK
- added U4: 7805n, symbol 7805n
Connections:
- net +3V3: now also U4.3 (VO)
- net +5V: now also Con11.1, U4.1 (VI)
- net GND: now also Con11.2, U4.2 (GND)
Changed lines of the file:
@@
 NeutralB
 $Comp
-L 7805 U4
-U 1 1 570B82C2
+L BARREL_JACK Con11
+U 1 1 5702E440
+P 1250 3100
+F 0 "Con11" H 1250 3350 50  0000 C CNN
+F 1 "BARREL_JACK" H 1250 2900 50  0000 C CNN
+F 2 "Connect:BARREL_JACK" H 1250 3100 50  0001 C CNN
+F 3 "" H 1250 3100 50  0000 C CNN
+	1    1250 3100
+	1    0    0    -1
+$EndComp
+$Comp
+L +5V #PWR040
+U 1 1 5702E5CD
+P 1700 2900
+F 0 "#PWR040" H 1700 2750 50  0001 C CNN
+F 1 "+5V" H 1700 3040 50  0000 C CNN
+F 2 "" H 1700 2900 50  0000 C CNN
+F 3 "" H 1700 2900 50  0000 C CNN
+	1    1700 2900
+	1    0    0    -1
+$EndComp
+Wire Wire Line
+	1700 2900 1700 3000
+Wire Wire Line
+	1700 3000 1550 3000
+$Comp
+L GND #PWR041
+U 1 1 5702E648
+P 1700 3300
+F 0 "#PWR041" H 1700 3050 50  0001 C CNN
+F 1 "GND" H 1700 3150 50  0000 C CNN
+F 2 "" H 1700 3300 50  0000 C CNN
+F 3 "" H 1700 3300 50  0000 C CNN
+	1    1700 3300
+	1    0    0    -1
+$EndComp
+Wire Wire Line
+	1700 3300 1700 3200
+Wire Wire Line
+	1700 3200 1550 3200
+$Comp
+L 7805n U4
+U 1 1 57034876
 P 3450 1500
 F 0 "U4" H 3600 1304 50  0000 C CNN
-F 1 "7805" H 3450 1700 50  0000 C CNN
-F 2 "TO_SOT_Packages_SMD:TO-252-2Lead" H 3450 1500 50  0001 C CNN
+F 1 "7805n" H 3450 1700 50  0000 C CNN
+F 2 "" H 3450 1500 50  0000 C CNN
 F 3 "" H 3450 1500 50  0000 C CNN
 	1    3450 1500
