File: DMX-Xi12/Power2.sch (KiCad schematic (older format))
At the start: 48 parts

Commit message: more schematic
Parts:
- removed U? (x6): Live, symbol Live
Connections:
- net labels added: Live10, Live11, Live12, Live7, Live8, Live9
Changed lines of the file:
@@
 Wire Wire Line
 	4800 1900 4800 2150
-$Comp
-L Live U?
-U 1 1 56B70101
-P 4800 800
-F 0 "U?" H 4850 850 60  0000 C CNN
-F 1 "Live" H 4800 1050 60  0000 C CNN
-F 2 "" H 4800 800 60  0000 C CNN
-F 3 "" H 4800 800 60  0000 C CNN
-	1    4800 800
-	1    0    0    -1
-$EndComp
 Connection ~ 4800 950
 Connection ~ 4800 2000
@@
 Wire Wire Line
 	4800 4000 4800 4250
-$Comp
-L Live U?
-U 1 1 56B70152
-P 4800 2900
-F 0 "U?" H 4850 2950 60  0000 C CNN
-F 1 "Live" H 4800 3150 60  0000 C CNN
-F 2 "" H 4800 2900 60  0000 C CNN
-F 3 "" H 4800 2900 60  0000 C CNN
-	1    4800 2900
-	1    0    0    -1
-$EndComp
 Connection ~ 4800 3050
 Connection ~ 4800 4100
@@
 Wire Wire Line
 	4800 6050 4800 6300
-$Comp
-L Live U?
-U 1 1 56B701A3
-P 4800 4950
-F 0 "U?" H 4850 5000 60  0000 C CNN
-F 1 "Live" H 4800 5200 60  0000 C CNN
-F 2 "" H 4800 4950 60  0000 C CNN
-F 3 "" H 4800 4950 60  0000 C CNN
-	1    4800 4950
-	1    0    0    -1
-$EndComp
 Connection ~ 4800 5100
 Connection ~ 4800 6150
@@
 Wire Wire Line
 	8800 1900 8800 2150
-$Comp
-L Live U?
-U 1 1 56B701F4
-P 8800 800
-F 0 "U?" H 8850 850 60  0000 C CNN
-F 1 "Live" H 8800 1050 60  0000 C CNN
-F 2 "" H 8800 800 60  0000 C CNN
-F 3 "" H 8800 800 60  0000 C CNN
-	1    8800 800
-	1    0    0    -1
-$EndComp
 Connection ~ 8800 950
 Connection ~ 8800 2000
@@
 Wire Wire Line
 	8800 4050 8800 4300
-$Comp
-L Live U?
-U 1 1 56B70245
-P 8800 2950
-F 0 "U?" H 8850 3000 60  0000 C CNN
-F 1 "Live" H 8800 3200 60  0000 C CNN
-F 2 "" H 8800 2950 60  0000 C CNN
-F 3 "" H 8800 2950 60  0000 C CNN
-	1    8800 2950
-	1    0    0    -1
-$EndComp
 Connection ~ 8800 3100
 Connection ~ 8800 4150
@@
 Wire Wire Line
 	8800 6000 8800 6250
-$Comp
-L Live U?
-U 1 1 56B70296
-P 8800 4900
-F 0 "U?" H 8850 4950 60  0000 C CNN
-F 1 "Live" H 8800 5150 60  0000 C CNN
-F 2 "" H 8800 4900 60  0000 C CNN
-F 3 "" H 8800 4900 60  0000 C CNN
-	1    8800 4900
-	1    0    0    -1
-$EndComp
 Connection ~ 8800 5050
 Connection ~ 8800 6100
@@
 	-1   0    0    1
 $EndComp
+Text Label 4800 800  1    60   ~ 0
+Live7
+Text Label 8800 800  1    60   ~ 0
+Live10
+Text Label 4800 2900 1    60   ~ 0
+Live8
+Text Label 8800 2950 1    60   ~ 0
+Live11
+Text Label 8800 4900 1    60   ~ 0
+Live12
+Text Label 4800 4950 1    60   ~ 0
+Live9
 $EndSCHEMATC

Commit message: made dlaw changes etc
Parts:
- removed C? (x6): 0.3u, symbol C
- removed R? (x6): 200R, symbol R
- removed R? (x6): 180R, symbol R
- removed R? (x6): 800R, symbol R
- removed U? (x6): AN-3003, symbol AN-3003
- removed U? (x6): BTA20, symbol BTA20
- removed U? (x6): Neutral, symbol Neutral
- added R? (x16): 200R, symbol R
- added R? (x16): 180R, symbol R
- added U? (x16): AN-3003, symbol AN-3003
- added U? (x16): BTA20, symbol BTA20
Connections:
- net labels added: CH17, CH18, CH19, CH20, CH21, CH22, CH23, CH24, CH25, CH26, CH27, CH28, CH29, CH30, CH31, CH32, Live17, Live18, Live19, Live20, Live21, Live22, Live23, Live24, Live25, Live26, Live27, Live28, Live29, Live30, Live31, Live32, NeutralB
- net labels removed: CH10, CH11, CH12, CH7, CH8, CH9, Live10, Live11, Live12, Live7, Live8, Live9
- wire segments 78 -> 144
- no-connect marks 12 -> 32

Commit message: working on pcb
Parts:
- R50, R51, R52, R53, R54, R55, R56, R57, R58, R59, R60, R61, R62, R63, R64, R65, R66, R67, R68, R69, R70, R71, R72, R73, R74, R75, R76, R77, R78, R79, R80, R81: renamed from R?; footprint (none) -> Resistors_SMD:R_0603
- U38, U39, U40, U41, U46, U47, U48, U49, U54, U55, U56, U57, U62, U63, U64, U65: renamed from U?; footprint (none) -> Housings_DIP:DIP-6_W7.62mm_LongPads
- U42, U43, U44, U45, U50, U51, U52, U53, U58, U59, U60, U61, U66, U67, U68, U69: renamed from U?; footprint (none) -> Power_Integrations:TO-220
Connections:
- net NeutralB renamed LiveB
